File: Attiny85_USB/Attiny85_USB/Attiny85_USB.kicad_pcb (KiCad board)
At the start: 2 copper layers, 40 x 12.2 mm, 12 parts, among them J1 Conn_01x04, J2 Conn_01x04, U1 ATtiny85-20S

Commit message: 7740
Parts:
- added H1: MountingHole, MountingHole:MountingHole_2.2mm_M2, F.Cu at (68.7, 110.6)
- added H2: MountingHole, MountingHole:MountingHole_2.2mm_M2, F.Cu at (104.5, 110.7)
- added H3: MountingHole, MountingHole:MountingHole_2.2mm_M2, F.Cu at (68.8, 117.4)
- added H4: MountingHole, MountingHole:MountingHole_2.2mm_M2, F.Cu at (104.5, 117.4)
- moved R3 39.0 mm to (93.4, 118.7)
- moved J2 35.9 mm to (98.8, 117.8), turned to 180 degrees
- moved R4 35.4 mm to (73.5, 113.9), turned to 180 degrees
- moved U2 34.2 mm to (56.6, 114.0)
- moved C1 32.8 mm to (87.0, 117.2), turned to 90 degrees
- moved R1 32.7 mm to (78.6, 116.6), turned to -90 degrees
- moved D2 32.5 mm to (74.2, 117.2), turned to 0 degrees
- moved D3 32.0 mm to (92.9, 115.9), turned to 0 degrees
- moved R2 31.0 mm to (78.6, 110.6), turned to -90 degrees
- moved U1 27.3 mm to (90.6, 111.3)
- moved J1 25.6 mm to (82.5, 110.1), turned to 0 degrees
- moved D1 25.0 mm to (74.2, 110.6), turned to 0 degrees
Routing:
- net GND: track 51.8 -> 8.97 mm, vias 0 -> 6
- net Net-(D1-K): track 22.8 -> 38.5 mm, vias 2 -> 0
- net +5V: track 44.2 -> 57.1 mm, vias 4 -> 0
- net Net-(J1-Pin_2): track 10.5 -> 21.2 mm
- net Net-(J1-Pin_1): track 15.5 -> 4.78 mm, vias 1 -> 0
- net Net-(J2-Pin_3): track 14.5 -> 5.69 mm, vias 1 -> 0
- net Net-(D2-K): track 36.0 -> 27.3 mm, vias 2 -> 0
- net Net-(J2-Pin_2): track 15.9 -> 21.8 mm
- net Net-(J1-Pin_3): track 16.3 -> 10.5 mm, vias 4 -> 0
- net Net-(J2-Pin_1): track 9.60 -> 7.51 mm
- net Net-(D3-A): track 4.80 -> 2.83 mm
- added copper zone on F.Cu, net +5V
- added copper zone on B.Cu, net GND
- added copper zone on F.Cu, net GND
Other:
- board size 40 x 12.2 mm -> 54.2 x 12.2 mm
