File: Attiny85_USB/Attiny85_USB/Attiny85_USB.kicad_sch (KiCad schematic)
At the start: 12 parts, among them J1 Conn_01x04, J2 Conn_01x04, U1 ATtiny85-20S

Commit message: 7740
Parts:
- added H1, H2, H3, H4: MountingHole, MountingHole:MountingHole_2.2mm_M2, symbol Mechanical:MountingHole
Changed lines of the file:
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@@
   (junction (at 177.8 128.27) (diameter 0) (color 0 0 0 0)
   )
+  (junction (at 209.55 128.27) (diameter 0) (color 0 0 0 0)
+  )
   (junction (at 163.83 128.27) (diameter 0) (color 0 0 0 0)
   )
   (junction (at 190.5 100.33) (diameter 0) (color 0 0 0 0)
   )
+  (junction (at 209.55 72.39) (diameter 0) (color 0 0 0 0)
+  )
   (junction (at 120.65 128.27) (diameter 0) (color 0 0 0 0)
   )
@@
   (junction (at 201.93 128.27) (diameter 0) (color 0 0 0 0)
   )
+  (wire (pts (xy 170.18 95.25) (xy 177.8 95.25))
+    (stroke (width 0) (type default))
+  )
+  (wire (pts (xy 190.5 90.17) (xy 190.5 100.33))
+    (stroke (width 0) (type default))
+  )
+  (wire (pts (xy 177.8 128.27) (xy 190.5 128.27))
+    (stroke (width 0) (type default))
+  )
+  (wire (pts (xy 120.65 128.27) (xy 163.83 128.27))
+    (stroke (width 0) (type default))
+  )
   (wire (pts (xy 120.65 115.57) (xy 120.65 128.27))
     (stroke (width 0) (type default))
   )
-  (wire (pts (xy 170.18 95.25) (xy 177.8 95.25))
-    (stroke (width 0) (type default))
-  )
-  (wire (pts (xy 190.5 90.17) (xy 190.5 100.33))
-    (stroke (width 0) (type default))
-  )
-  (wire (pts (xy 177.8 128.27) (xy 190.5 128.27))
-    (stroke (width 0) (type default))
-  )
-  (wire (pts (xy 120.65 128.27) (xy 163.83 128.27))
+  (wire (pts (xy 152.4 116.84) (xy 152.4 100.33))
+    (stroke (width 0) (type default))
+  )
+  (wire (pts (xy 163.83 116.84) (xy 163.83 128.27))
+    (stroke (width 0) (type default))
+  )
+  (wire (pts (xy 212.09 105.41) (xy 209.55 105.41))
+    (stroke (width 0) (type default))
+  )
+  (wire (pts (xy 152.4 100.33) (xy 135.89 100.33))
+    (stroke (width 0) (type default))
+  )
+  (wire (pts (xy 90.17 99.06) (xy 90.17 72.39))
+    (stroke (width 0) (type default))
+  )
+  (wire (pts (xy 209.55 97.79) (xy 209.55 72.39))
+    (stroke (width 0) (type default))
+  )
+  (wire (pts (xy 190.5 100.33) (xy 212.09 100.33))
+    (stroke (width 0) (type default))
+  )
+  (wire (pts (xy 154.94 95.25) (xy 135.89 95.25))
+    (stroke (width 0) (type default))
+  )
+  (wire (pts (xy 190.5 72.39) (xy 140.97 72.39))
+    (stroke (width 0) (type default))
+  )
+  (wire (pts (xy 190.5 118.11) (xy 190.5 128.27))
+    (stroke (width 0) (type default))
+  )
+  (wire (pts (xy 201.93 128.27) (xy 190.5 128.27))
+    (stroke (width 0) (type default))
+  )
+  (wire (pts (xy 90.17 128.27) (xy 90.17 104.14))
+    (stroke (width 0) (type default))
+  )
+  (wire (pts (xy 201.93 102.87) (xy 212.09 102.87))
+    (stroke (width 0) (type default))
+  )
+  (wire (pts (xy 209.55 72.39) (xy 190.5 72.39))
+    (stroke (width 0) (type default))
+  )
+  (wire (pts (xy 212.09 97.79) (xy 209.55 97.79))
+    (stroke (width 0) (type default))
+  )
+  (wire (pts (xy 135.89 102.87) (xy 154.94 102.87))
     (stroke (width 0) (type default))
   )
@@
     (stroke (width 0) (type default))
   )
-  (wire (pts (xy 152.4 116.84) (xy 152.4 100.33))
-    (stroke (width 0) (type default))
-  )
-  (wire (pts (xy 163.83 116.84) (xy 163.83 128.27))
-    (stroke (width 0) (type default))
-  )
-  (wire (pts (xy 212.09 105.41) (xy 209.55 105.41))
-    (stroke (width 0) (type default))
-  )
-  (wire (pts (xy 152.4 100.33) (xy 135.89 100.33))
-    (stroke (width 0) (type default))
-  )
-  (wire (pts (xy 90.17 99.06) (xy 90.17 72.39))
-    (stroke (width 0) (type default))
-  )
-  (wire (pts (xy 209.55 97.79) (xy 209.55 72.39))
-    (stroke (width 0) (type default))
-  )
-  (wire (pts (xy 190.5 100.33) (xy 212.09 100.33))
-    (stroke (width 0) (type default))
-  )
-  (wire (pts (xy 154.94 95.25) (xy 135.89 95.25))
-    (stroke (width 0) (type default))
-  )
-  (wire (pts (xy 190.5 72.39) (xy 140.97 72.39))
-    (stroke (width 0) (type default))
-  )
-  (wire (pts (xy 190.5 118.11) (xy 190.5 128.27))
-    (stroke (width 0) (type default))
-  )
-  (wire (pts (xy 201.93 128.27) (xy 190.5 128.27))
-    (stroke (width 0) (type default))
-  )
-  (wire (pts (xy 90.17 128.27) (xy 90.17 104.14))
-    (stroke (width 0) (type default))
-  )
-  (wire (pts (xy 201.93 102.87) (xy 212.09 102.87))
-    (stroke (width 0) (type default))
-  )
-  (wire (pts (xy 209.55 72.39) (xy 190.5 72.39))
-    (stroke (width 0) (type default))
-  )
-  (wire (pts (xy 212.09 97.79) (xy 209.55 97.79))
-    (stroke (width 0) (type default))
-  )
-  (wire (pts (xy 135.89 102.87) (xy 154.94 102.87))
-    (stroke (width 0) (type default))
-  )
   (wire (pts (xy 190.5 82.55) (xy 190.5 72.39))
     (stroke (width 0) (type default))
@@
     (stroke (width 0) (type default))
   )
+  (symbol (lib_id "power:PWR_FLAG") (at 209.55 72.39 0) (unit 1)
+    (in_bom yes) (on_board yes) (dnp no) (fields_autoplaced)
+    (property "Reference" "#FLG01" (at 209.55 70.485 0)
+      (effects (font (size 1.27 1.27)) hide)
+    )
+    (property "Value" "PWR_FLAG" (at 209.55 68.58 0)
+      (effects (font (size 1.27 1.27)))
+    )
+    (property "Footprint" "" (at 209.55 72.39 0)
+      (effects (font (size 1.27 1.27)) hide)
+    )
+    (property "Datasheet" "~" (at 209.55 72.39 0)
+      (effects (font (size 1.27 1.27)) hide)
+    )
+    (pin "1")
+    (instances
+      (project "Attiny85_USB"
+        (path "/68905119-dc09-4750-af87-5d11388f557f"
+          (reference "#FLG01") (unit 1)
+        )
+      )
+    )
+  )
   (symbol (lib_id "Device:R") (at 190.5 86.36 0) (unit 1)
     (in_bom yes) (on_board yes) (dnp no) (fields_autoplaced)
@@
         (path "/68905119-dc09-4750-af87-5d11388f557f"
           (reference "R4") (unit 1)
+        )
+      )
+    )
+  )
+  (symbol (lib_id "Mechanical:MountingHole") (at 242.57 96.52 0) (unit 1)
+    (in_bom yes) (on_board yes) (dnp no) (fields_autoplaced)
+    (property "Reference" "H3" (at 245.11 95.885 0)
+      (effects (font (size 1.27 1.27)) (justify left))
+    )
+    (property "Value" "MountingHole" (at 245.11 98.425 0)
+      (effects (font (size 1.27 1.27)) (justify left))
+    )
+    (property "Footprint" "MountingHole:MountingHole_2.2mm_M2" (at 242.57 96.52 0)
+      (effects (font (size 1.27 1.27)) hide)
+    )
+    (property "Datasheet" "~" (at 242.57 96.52 0)
+      (effects (font (size 1.27 1.27)) hide)
+    )
+    (instances
+      (project "Attiny85_USB"
+        (path "/68905119-dc09-4750-af87-5d11388f557f"
+          (reference "H3") (unit 1)
         )
       )
@@
         (path "/68905119-dc09-4750-af87-5d11388f557f"
           (reference "R1") (unit 1)
+        )
+      )
+    )
+  )
+  (symbol (lib_id "Mechanical:MountingHole") (at 242.57 90.17 0) (unit 1)
+    (in_bom yes) (on_board yes) (dnp no) (fields_autoplaced)
+    (property "Reference" "H2" (at 245.11 89.535 0)
+      (effects (font (size 1.27 1.27)) (justify left))
+    )
+    (property "Value" "MountingHole" (at 245.11 92.075 0)
+      (effects (font (size 1.27 1.27)) (justify left))
+    )
+    (property "Footprint" "MountingHole:MountingHole_2.2mm_M2" (at 242.57 90.17 0)
+      (effects (font (size 1.27 1.27)) hide)
+    )
+    (property "Datasheet" "~" (at 242.57 90.17 0)
+      (effects (font (size 1.27 1.27)) hide)
+    )
+    (instances
+      (project "Attiny85_USB"
+        (path "/68905119-dc09-4750-af87-5d11388f557f"
+          (reference "H2") (unit 1)
+        )
+      )
+    )
+  )
+  (symbol (lib_id "Mechanical:MountingHole") (at 242.57 102.87 0) (unit 1)
+    (in_bom yes) (on_board yes) (dnp no) (fields_autoplaced)
+    (property "Reference" "H4" (at 245.11 102.235 0)
+      (effects (font (size 1.27 1.27)) (justify left))
+    )
+    (property "Value" "MountingHole" (at 245.11 104.775 0)
+      (effects (font (size 1.27 1.27)) (justify left))
+    )
+    (property "Footprint" "MountingHole:MountingHole_2.2mm_M2" (at 242.57 102.87 0)
+      (effects (font (size 1.27 1.27)) hide)
+    )
+    (property "Datasheet" "~" (at 242.57 102.87 0)
+      (effects (font (size 1.27 1.27)) hide)
+    )
+    (instances
+      (project "Attiny85_USB"
+        (path "/68905119-dc09-4750-af87-5d11388f557f"
+          (reference "H4") (unit 1)
+        )
+      )
+    )
+  )
+  (symbol (lib_id "power:PWR_FLAG") (at 209.55 128.27 180) (unit 1)
+    (in_bom yes) (on_board yes) (dnp no) (fields_autoplaced)
+    (property "Reference" "#FLG02" (at 209.55 130.175 0)
+      (effects (font (size 1.27 1.27)) hide)
+    )
+    (property "Value" "PWR_FLAG" (at 209.55 133.35 0)
+      (effects (font (size 1.27 1.27)))
+    )
+    (property "Footprint" "" (at 209.55 128.27 0)
+      (effects (font (size 1.27 1.27)) hide)
+    )
+    (property "Datasheet" "~" (at 209.55 128.27 0)
+      (effects (font (size 1.27 1.27)) hide)
+    )
+    (pin "1")
+    (instances
+      (project "Attiny85_USB"
+        (path "/68905119-dc09-4750-af87-5d11388f557f"
+          (reference "#FLG02") (unit 1)
         )
       )
@@
         )
       )
+    )
+  )
+  (symbol (lib_id "Mechanical:MountingHole") (at 242.57 83.82 0) (unit 1)
+    (in_bom yes) (on_board yes) (dnp no) (fields_autoplaced)
+    (property "Reference" "H1" (at 245.11 83.185 0)
+      (effects (font (size 1.27 1.27)) (justify left))
+    )
+    (property "Value" "MountingHole" (at 245.11 85.725 0)
+      (effects (font (size 1.27 1.27)) (justify left))
+    )
+    (property "Footprint" "MountingHole:MountingHole_2.2mm_M2" (at 242.57 83.82 0)
+      (effects (font (size 1.27 1.27)) hide)
+    )
+    (property "Datasheet" "~" (at 242.57 83.82 0)
+      (effects (font (size 1.27 1.27)) hide)
+    )
+    (instances
+      (project "Attiny85_USB"
+        (path "/68905119-dc09-4750-af87-5d11388f557f"
+          (reference "H1") (unit 1)
+        )
+      )
