File: STM32F405RGT6/STM32F405RGT6/STM32F405RGT6.kicad_sch (KiCad schematic)
At the start: 18 parts, among them SW1 SW_SPDT, U1 STM32F405RGT6, Y1 16MHz

Commit message: Dell 7740
Parts:
- added D1: LED_Small, LED_SMD:LED_0603_1608Metric, symbol Device:LED_Small
- added H1, H2, H3, H4: MountingHole_Pad, MountingHole:MountingHole_4.3mm_M4_Pad_Via, symbol Mechanical:MountingHole_Pad
- added J1: Screw_Terminal_01x03, TerminalBlock_Phoenix:TerminalBlock_Phoenix_PT-1,5-3-5.0-H_1x03_P5.00mm_Horizontal, symbol Connector:Screw_Terminal_01x03
- added J2: SWD, Connector_PinSocket_1.27mm:PinSocket_2x05_P1.27mm_Vertical, symbol Connector_Generic:Conn_02x05_Odd_Even
- added J3: I2C1, Connector_Molex:Molex_PicoBlade_53048-0410_1x04_P1.25mm_Horizontal, symbol Connector_Generic:Conn_01x04
- added J4: USART3, Connector_Molex:Molex_PicoBlade_53048-0410_1x04_P1.25mm_Horizontal, symbol Connector_Generic:Conn_01x04
- added J5: USB_B_Micro, Connector_USB:USB_Micro-B_Amphenol_10118193-0002LF_Horizontal, symbol Connector:USB_B_Micro
- added R3: 1k5, Resistor_SMD:R_0603_1608Metric, symbol Device:R_Small
- added R4: 22, Resistor_SMD:R_0603_1608Metric, symbol Device:R_Small
- added R5, R6: 2K2, Resistor_SMD:R_0603_1608Metric, symbol Device:R_Small
- added U2: USBLC6-2SC6, Package_TO_SOT_SMD:SOT-23-6, symbol Power_Protection:USBLC6-2SC6
- C1, C10, C2, C3: footprint (none) -> Capacitor_SMD:C_0603_1608Metric
- C11, C12, C4, C5, C6, C7, C8, C9: footprint (none) -> Capacitor_SMD:C_0402_1005Metric
- L1: footprint (none) -> Inductor_SMD:L_0402_1005Metric
- R1, R2: footprint (none) -> Resistor_SMD:R_0603_1608Metric
- SW1: footprint (none) -> Button_Switch_SMD:SW_SPDT_PCM12
- Y1: footprint (none) -> Crystal:Crystal_SMD_3225-4Pin_3.2x2.5mm
Connections:
- net +3.3V: now also J1.1 (Pin_1), J3.1 (Pin_1), J4.1 (Pin_1), R5.2, R6.2
- net +3.3VA: now also J1.2 (Pin_2), J2.1 (Pin_1)
- net GND: now also H1.1, H2.1, H3.1, H4.1, J1.3 (Pin_3), J2.3 (Pin_3), J2.5 (Pin_5), J2.9 (Pin_9), J3.4 (Pin_4), J4.4 (Pin_4), J5.5 (GND), R3.1, U2.2 (GND)
- net I2C1_SCL: now also J3.2 (Pin_2), R6.1
- net I2C1_SDA: now also J3.3 (Pin_3), R5.1
- net LED_STATUS: now also D1.2 (A)
- net NRST: now also J2.10 (Pin_10)
- net SWCLK: now also J2.4 (Pin_4)
- net SWDIO: now also R4.1
- net USART3_RX: now also J4.3 (Pin_3)
- net USART3_TX: now also J4.2 (Pin_2)
- net USB_D+: now also U2.4 (I/O2)
- net USB_D-: now also U2.6 (I/O1)
- net SWD renamed SWO
- net SWO: now also J2.6 (Pin_6)
- new net: J2.2 (Pin_2), R4.2
- new net: D1.1 (K), R3.2
- new net +5V: J5.1 (VBUS), U2.5 (VBUS)
- new net USB_CONN_D+: J5.3 (D+), U2.3 (I/O2)
- new net USB_CONN_D-: J5.2 (D-), U2.1 (I/O1)
- no-connect marks 39 -> 43
