File: qPCR Modules/qPCR Module/qPCR Module.kicad_sch (KiCad schematic)
At the start: 2 parts, among them Q1 BC337, U1 ESP32-S3-DevKitC

Commit message: Dell 7740
Parts:
- added D1: LED, symbol Device:LED
- added J1: Logic Parts, symbol Connector_Generic:Conn_01x03
- added J2: TEC Controller, symbol Connector_Generic:Conn_01x02
- added PE1: PeltierElement, symbol Device:PeltierElement
- added R1, R2: 2k2, symbol Device:R
- added TH1: NTC_Sink Temp, symbol Device:Thermistor_NTC
- added TH2: PT100_Reactor Temp, symbol Sensor_Temperature:PT100
- added U2: ~, symbol Hai_Library:VEML7700
- added U3: ~, symbol Hai_Library:TEC_1091
Connections:
- net +3.3V: now reaches U1.1 (3V3), U1.2 (3V3)
- net +3.3V: now also J1.1 (Pin_1)
- net UART1_RX: now reaches U1.16 (GPIO10/ADC1_CH9)
- net UART1_RX: now also U3.8 (RS232_TTL_TX)
- net UART1_TX: now reaches U1.17 (GPIO11/ADC2_CH0)
- net UART1_TX: now also U3.7 (RS232_TTL_RX)
- net +5V: now reaches U1.21 (5V)
- net +5V: now also D1.2 (A), J1.3 (Pin_3), U2.1 (Vin)
- net Emission Led: now reaches U1.4 (GPIO4/ADC1_CH3)
- net Emission Led: now also R1.1
- net SDA: now reaches U1.8 (GPIO15/ADC2_CH4/32K_P)
- net SDA: now also U2.5 (SDA)
- net SCL: now reaches U1.9 (GPIO16/ADC2_CH5/32K_N)
- net SCL: now also U2.4 (SCL)
- net at Q1.1 (C): now also D1.1 (K)
- net at Q1.2 (B): now also R1.2
- net at Q1.3 (E): now also R2.2
- new net: PE1.1, U3.1 (VIN)
- new net: TH2.1, U3.10 (RS485_B2_(D-),_CANL), U3.8 (RS232_TTL_TX)
- new net: PE1.2, U3.2 (OUT-)
- new net: TH1.1, U3.4 (SINK_To_B)
- new net: TH1.2, U3.5 (SINK_To_A)
- new net: TH2.2, U3.7 (RS232_TTL_RX), U3.9 (RS485_A2_(D+),_CANH)
- new net +24V: J2.2 (Pin_2), U3.1 (VIN)
- new net GND: J1.2 (Pin_2), J2.1 (Pin_1), R2.1, U2.3 (GND), U3.2 (OUT-)
- no-connect marks 0 -> 9
Other:
- note added: "Control Emission Led"
- note added: "Controller Unit"
- note added: "Emission fliter"
- note added: "Excitation Filter"
- note added: "Fluorescence Measurement"
- note added: "Power Input"
- note added: "Proposed Design of qPCR System"
- note added: "Thermal control block"
- title: (none) -> qPCR System
- moved on the sheet: Q1, U1

Commit message: Dell 7740
Connections:
- net UART2_TX: now reaches U1.40 (GPIO2/ADC1_CH1)
- net UART2_RX: now reaches U1.41 (GPIO1/ADC1_CH0)
- net at U3.10 (RS485_B2_(D-),_CANL): now also TH2.1, U3.8 (RS232_TTL_TX)
- net at U3.4 (SINK_To_B): now also TH1.1
- net at U3.5 (SINK_To_A): now also TH1.2
- new net: TH2.2, U3.7 (RS232_TTL_RX), U3.9 (RS485_A2_(D+),_CANH)
- now unconnected: U3.9 (RS485_A2_(D+),_CANH)

Commit message: Dell 7740
Parts:
- R1: value 2k2 -> 3k3
- R2: value 2k2 -> 47
Connections:
- net +5V: now also R2.2; no longer D1.2 (A)
- net GND: now also Q1.3 (E); no longer R2.1
- net at U3.10 (RS485_B2_(D-),_CANL): now also TH2.1, U3.8 (RS232_TTL_TX)
- net at U3.4 (SINK_To_B): now also TH1.1
- net at U3.5 (SINK_To_A): now also TH1.2
- new net: D1.2 (A), R2.1
- new net: TH2.2, U3.7 (RS232_TTL_RX), U3.9 (RS485_A2_(D+),_CANH)
- now unconnected: U3.9 (RS485_A2_(D+),_CANH)
Other:
- note added: "I_Led = 30mA"
- moved on the sheet: D1, Q1, R1
